Commit message: Update _d435.urdf.xacro

File: realsense2_description/urdf/_d435.urdf.xacro (robot description, xacro)
@@ -11,5 +11,4 @@
   <xacro:include filename="$(find realsense2_description)/urdf/_usb_plug.urdf.xacro" />
   <xacro:macro name="sensor_d435" params="parent *origin name:=camera use_nominal_extrinsics:=false">
-    <xacro:arg name="add_plug" default="false" />
     <xacro:property name="M_PI" value="3.1415926535897931" />
     <!-- The following values are approximate, and the camera node
@@ -65,5 +64,5 @@
       <inertial>
         <!-- The following are not reliable values, and should not be used for modeling -->
-        <mass value="0.072" />
+        <mass value="0.564" />
         <origin xyz="0 0 0" />
         <inertia ixx="0.003881243" ixy="0.0" ixz="0.0" iyy="0.000498940" iyz="0.0" izz="0.003879257" />
@@ -125,9 +124,10 @@
       <link name="${name}_color_optical_frame"/>
     </xacro:if>
-    <xacro:if value="$(arg add_plug)">
+    <!-- I was getting the error shown below, so I just uncommented this xacro portion since I'm using ROS Melodic  -->
+    <!-- <xacro:if value="$(arg add_plug)">
       <xacro:usb_plug parent="${name}_link">
         <origin xyz="${d435_cam_mount_from_center_offset - 0.02095} ${-d435_cam_depth_py - 0.0353} 0" rpy="0 0 0"/>
       </xacro:usb_plug>
-    </xacro:if>
+    </xacro:if> -->
   </xacro:macro>
 </robot>
